File: cellar/General_purpose.sch (KiCad schematic (older format))
At the start: 21 parts, among them Q11 IRLML6344TRPBF

Commit message: Replaced wirepads by phoenix connectors.
Parts:
- removed W30: SWITCH0+, Pads:wirepad_hole_2.2x1mm, symbol pads:WirePad
- removed W31: SWITCH0_GND, Pads:wirepad_hole_2.2x1mm, symbol pads:WirePad
- removed W32: ADC1, symbol pads:WirePad
- removed W33: ADC2, symbol pads:WirePad
- removed W34: ADC3, symbol pads:WirePad
- C26: renamed from C28; footprint (none) -> Capacitor_SMD:C_0805_2012Metric_Pad1.15x1.40mm_HandSolder
- C27: renamed from C29; footprint (none) -> Capacitor_SMD:C_0805_2012Metric_Pad1.15x1.40mm_HandSolder
- C28: renamed from C30; footprint (none) -> Capacitor_SMD:C_0805_2012Metric_Pad1.15x1.40mm_HandSolder
- D14: Farnell 5790852 -> 2251490; Ref HSMG-C170 -> VLMTG1300-GS08
- renumbered D12 to D13, R47 to R50, R48 to R51, R49 to R52, R50 to R53
Connections:
- net labels added: SWITCH0+, SWITCH0_GND
Changed lines of the file:
@@
 P 2500 3300
 AR Path="/5BCDDEA6/5BEA4E3D" Ref="#PWR?"  Part="1"
-AR Path="/5BEA0F8F/5BEA4E3D" Ref="#PWR044"  Part="1"
-F 0 "#PWR044" H 2500 3050 50  0001 C CNN
+AR Path="/5BEA0F8F/5BEA4E3D" Ref="#PWR054"  Part="1"
+F 0 "#PWR054" H 2500 3050 50  0001 C CNN
 F 1 "GND" H 2505 3127 50  0000 C CNN
 F 2 "" H 2500 3300 50  0001 C CNN
@@
 P 2300 2950
 AR Path="/5BCDDEA6/5BEA4E43" Ref="R?"  Part="1"
-AR Path="/5BEA0F8F/5BEA4E43" Ref="R49"  Part="1"
-F 0 "R49" H 2230 2904 50  0000 R CNN
+AR Path="/5BEA0F8F/5BEA4E43" Ref="R52"  Part="1"
+F 0 "R52" H 2230 2904 50  0000 R CNN
 F 1 "10k" H 2230 2995 50  0000 R CNN
 F 2 "" V 2230 2950 50  0001 C CNN
@@
 P 1100 1350
 AR Path="/5BCDDEA6/5BEA4E59" Ref="#PWR?"  Part="1"
-AR Path="/5BEA0F8F/5BEA4E59" Ref="#PWR042"  Part="1"
-F 0 "#PWR042" H 1100 1200 50  0001 C CNN
+AR Path="/5BEA0F8F/5BEA4E59" Ref="#PWR052"  Part="1"
+F 0 "#PWR052" H 1100 1200 50  0001 C CNN
 F 1 "+12V" H 1115 1523 50  0000 C CNN
 F 2 "" H 1100 1350 50  0001 C CNN
@@
 P 1400 1350
 AR Path="/5BCDDEA6/5BEA4E5F" Ref="#PWR?"  Part="1"
-AR Path="/5BEA0F8F/5BEA4E5F" Ref="#PWR043"  Part="1"
-F 0 "#PWR043" H 1400 1200 50  0001 C CNN
+AR Path="/5BEA0F8F/5BEA4E5F" Ref="#PWR053"  Part="1"
+F 0 "#PWR053" H 1400 1200 50  0001 C CNN
 F 1 "+5V" H 1415 1523 50  0000 C CNN
 F 2 "" H 1400 1350 50  0001 C CNN
@@
 P 1100 1650
 AR Path="/5BCDDEA6/5BEA4E65" Ref="R?"  Part="1"
-AR Path="/5BEA0F8F/5BEA4E65" Ref="R47"  Part="1"
-F 0 "R47" H 1030 1604 50  0000 R CNN
+AR Path="/5BEA0F8F/5BEA4E65" Ref="R50"  Part="1"
+F 0 "R50" H 1030 1604 50  0000 R CNN
 F 1 "0" H 1030 1695 50  0000 R CNN
 F 2 "" V 1030 1650 50  0001 C CNN
@@
 P 1400 1650
 AR Path="/5BCDDEA6/5BEA4E6C" Ref="R?"  Part="1"
-AR Path="/5BEA0F8F/5BEA4E6C" Ref="R48"  Part="1"
-F 0 "R48" H 1470 1696 50  0000 L CNN
+AR Path="/5BEA0F8F/5BEA4E6C" Ref="R51"  Part="1"
+F 0 "R51" H 1470 1696 50  0000 L CNN
 F 1 "0" H 1470 1605 50  0000 L CNN
 F 2 "" V 1330 1650 50  0001 C CNN
@@
 Connection ~ 2700 2050
 Wire Wire Line
-	2700 2050 2700 1400
-Wire Wire Line
-	1800 2050 1800 1400
+	2700 2050 2700 1650
+Wire Wire Line
+	1800 2050 1800 1650
 Connection ~ 1800 2050
 Wire Wire Line
 	1800 2050 2100 2050
-$Comp
-L pads:WirePad W?
-U 1 1 5BEA4E82
-P 1800 1400
-AR Path="/5BCDDEA6/5BEA4E82" Ref="W?"  Part="1"
-AR Path="/5BEA0F8F/5BEA4E82" Ref="W30"  Part="1"
-F 0 "W30" H 1722 1285 50  0000 R CNN
-F 1 "SWITCH0+" H 1722 1376 50  0000 R CNN
-F 2 "Pads:wirepad_hole_2.2x1mm" H 1800 1400 50  0001 C CNN
-F 3 "" H 1800 1400 50  0001 C CNN
-	1    1800 1400
-	-1   0    0    1
-$EndComp
-$Comp
-L pads:WirePad W?
-U 1 1 5BEA4E89
-P 2700 1400
-AR Path="/5BCDDEA6/5BEA4E89" Ref="W?"  Part="1"
-AR Path="/5BEA0F8F/5BEA4E89" Ref="W31"  Part="1"
-F 0 "W31" H 2622 1285 50  0000 R CNN
-F 1 "SWITCH0_GND" H 2622 1376 50  0000 R CNN
-F 2 "Pads:wirepad_hole_2.2x1mm" H 2700 1400 50  0001 C CNN
-F 3 "" H 2700 1400 50  0001 C CNN
-	1    2700 1400
-	-1   0    0    1
-$EndComp
 $Comp
 L Device:D D?
@@
 AR Path="/5BCDDEA3/5BEA4E92" Ref="D?"  Part="1"
 AR Path="/5BCDDEA6/5BEA4E92" Ref="D?"  Part="1"
-AR Path="/5BEA0F8F/5BEA4E92" Ref="D12"  Part="1"
-F 0 "D12" H 2250 2266 50  0000 C CNN
+AR Path="/5BEA0F8F/5BEA4E92" Ref="D13"  Part="1"
+F 0 "D13" H 2250 2266 50  0000 C CNN
 F 1 "SBR160S23-7" H 2250 2175 50  0000 C CNN
 F 2 "" H 2250 2050 50  0001 C CNN
@@
 F 2 "" H 3450 1500 50  0001 C CNN
 F 3 "~" H 3450 1500 50  0001 C CNN
-F 4 "5790852" H -6550 -2650 50  0001 C CNN "Farnell"
-F 5 "HSMG-C170" H -6550 -2650 50  0001 C CNN "Ref"
+F 4 "2251490" H -6550 -2650 50  0001 C CNN "Farnell"
+F 5 "VLMTG1300-GS08" H -6550 -2650 50  0001 C CNN "Ref"
 	1    3450 1500
 	0    -1   -1   0
@@
 P 3450 1300
 AR Path="/5BCDDEA6/5BEA4EA9" Ref="#PWR?"  Part="1"
-AR Path="/5BEA0F8F/5BEA4EA9" Ref="#PWR056"  Part="1"
-F 0 "#PWR056" H 3450 1150 50  0001 C CNN
+AR Path="/5BEA0F8F/5BEA4EA9" Ref="#PWR055"  Part="1"
+F 0 "#PWR055" H 3450 1150 50  0001 C CNN
 F 1 "+5V" H 3465 1473 50  0000 C CNN
 F 2 "" H 3450 1300 50  0001 C CNN
@@
 P 3450 1850
 AR Path="/5BCDDEA6/5BEA4EB1" Ref="R?"  Part="1"
-AR Path="/5BEA0F8F/5BEA4EB1" Ref="R50"  Part="1"
-F 0 "R50" H 3380 1804 50  0000 R CNN
+AR Path="/5BEA0F8F/5BEA4EB1" Ref="R53"  Part="1"
+F 0 "R53" H 3380 1804 50  0000 R CNN
 F 1 "1k" H 3380 1895 50  0000 R CNN
 F 2 "" V 3380 1850 50  0001 C CNN
@@
 P 6000 2500
 AR Path="/5BCDDEA9/5BEA6F66" Ref="C?"  Part="1"
-AR Path="/5BEA0F8F/5BEA6F66" Ref="C28"  Part="1"
-F 0 "C28" H 6115 2546 50  0000 L CNN
+AR Path="/5BEA0F8F/5BEA6F66" Ref="C26"  Part="1"
+F 0 "C26" H 6115 2546 50  0000 L CNN
 F 1 "UNKN" H 6050 2400 50  0000 L CNN
-F 2 "" H 6038 2350 50  0001 C CNN
+F 2 "Capacitor_SMD:C_0805_2012Metric_Pad1.15x1.40mm_HandSolder" H 6038 2350 50  0001 C CNN
 F 3 "~" H 6000 2500 50  0001 C CNN
 	1    6000 2500
@@
 P 5650 2850
 AR Path="/5BCDDEA9/5BEA6F77" Ref="#PWR?"  Part="1"
-AR Path="/5BEA0F8F/5BEA6F77" Ref="#PWR057"  Part="1"
-F 0 "#PWR057" H 5650 2600 50  0001 C CNN
+AR Path="/5BEA0F8F/5BEA6F77" Ref="#PWR056"  Part="1"
+F 0 "#PWR056" H 5650 2600 50  0001 C CNN
 F 1 "GND" H 5655 2677 50  0000 C CNN
 F 2 "" H 5650 2850 50  0001 C CNN
@@
 Text GLabel 6100 2200 2    50   Output ~ 0
 ADC1
-$Comp
-L pads:WirePad W?
-U 1 1 5BEA6F7E
-P 5650 1600
-AR Path="/5BCDDEA9/5BEA6F7E" Ref="W?"  Part="1"
-AR Path="/5BEA0F8F/5BEA6F7E" Ref="W32"  Part="1"
-F 0 "W32" H 5572 1485 50  0000 R CNN
-F 1 "ADC1" H 5572 1576 50  0000 R CNN
-F 2 "" H 5650 1600 50  0001 C CNN
-F 3 "" H 5650 1600 50  0001 C CNN
-	1    5650 1600
-	-1   0    0    1
-$EndComp
 Wire Wire Line
 	5650 2050 5650 2200
@@
 P 7150 2500
 AR Path="/5BCDDEA9/5BEA6F96" Ref="C?"  Part="1"
-AR Path="/5BEA0F8F/5BEA6F96" Ref="C29"  Part="1"
-F 0 "C29" H 7265 2546 50  0000 L CNN
+AR Path="/5BEA0F8F/5BEA6F96" Ref="C27"  Part="1"
+F 0 "C27" H 7265 2546 50  0000 L CNN
 F 1 "UNKN" H 7200 2400 50  0000 L CNN
-F 2 "" H 7188 2350 50  0001 C CNN
+F 2 "Capacitor_SMD:C_0805_2012Metric_Pad1.15x1.40mm_HandSolder" H 7188 2350 50  0001 C CNN
 F 3 "~" H 7150 2500 50  0001 C CNN
 	1    7150 2500
@@
 P 6800 2850
 AR Path="/5BCDDEA9/5BEA6FA7" Ref="#PWR?"  Part="1"
-AR Path="/5BEA0F8F/5BEA6FA7" Ref="#PWR058"  Part="1"
-F 0 "#PWR058" H 6800 2600 50  0001 C CNN
+AR Path="/5BEA0F8F/5BEA6FA7" Ref="#PWR057"  Part="1"
+F 0 "#PWR057" H 6800 2600 50  0001 C CNN
 F 1 "GND" H 6805 2677 50  0000 C CNN
 F 2 "" H 6800 2850 50  0001 C CNN
@@
 Text GLabel 7250 2200 2    50   Output ~ 0
 ADC2
-$Comp
-L pads:WirePad W?
-U 1 1 5BEA6FAE
-P 6800 1600
-AR Path="/5BCDDEA9/5BEA6FAE" Ref="W?"  Part="1"
-AR Path="/5BEA0F8F/5BEA6FAE" Ref="W33"  Part="1"
-F 0 "W33" H 6722 1485 50  0000 R CNN
-F 1 "ADC2" H 6722 1576 50  0000 R CNN
-F 2 "" H 6800 1600 50  0001 C CNN
-F 3 "" H 6800 1600 50  0001 C CNN
-	1    6800 1600
-	-1   0    0    1
-$EndComp
 Wire Wire Line
 	6800 2050 6800 2200
@@
 P 8250 2500
 AR Path="/5BCDDEA9/5BEA6FC6" Ref="C?"  Part="1"
-AR Path="/5BEA0F8F/5BEA6FC6" Ref="C30"  Part="1"
-F 0 "C30" H 8365 2546 50  0000 L CNN
+AR Path="/5BEA0F8F/5BEA6FC6" Ref="C28"  Part="1"
+F 0 "C28" H 8365 2546 50  0000 L CNN
 F 1 "UNKN" H 8300 2400 50  0000 L CNN
-F 2 "" H 8288 2350 50  0001 C CNN
+F 2 "Capacitor_SMD:C_0805_2012Metric_Pad1.15x1.40mm_HandSolder" H 8288 2350 50  0001 C CNN
 F 3 "~" H 8250 2500 50  0001 C CNN
 	1    8250 2500
@@
 P 7900 2850
 AR Path="/5BCDDEA9/5BEA6FD7" Ref="#PWR?"  Part="1"
-AR Path="/5BEA0F8F/5BEA6FD7" Ref="#PWR059"  Part="1"
-F 0 "#PWR059" H 7900 2600 50  0001 C CNN
+AR Path="/5BEA0F8F/5BEA6FD7" Ref="#PWR058"  Part="1"
+F 0 "#PWR058" H 7900 2600 50  0001 C CNN
 F 1 "GND" H 7905 2677 50  0000 C CNN
 F 2 "" H 7900 2850 50  0001 C CNN
@@
 Text GLabel 8350 2200 2    50   Output ~ 0
 ADC3
-$Comp
-L pads:WirePad W?
-U 1 1 5BEA6FDE
-P 7900 1600
-AR Path="/5BCDDEA9/5BEA6FDE" Ref="W?"  Part="1"
-AR Path="/5BEA0F8F/5BEA6FDE" Ref="W34"  Part="1"
-F 0 "W34" H 7822 1485 50  0000 R CNN
-F 1 "ADC3" H 7822 1576 50  0000 R CNN
-F 2 "" H 7900 1600 50  0001 C CNN
-F 3 "" H 7900 1600 50  0001 C CNN
-	1    7900 1600
-	-1   0    0    1
-$EndComp
 Wire Wire Line
 	7900 2050 7900 2200
@@
 Text Notes 6700 1150 0    118  ~ 24
 ADCs
+Text GLabel 1800 1650 1    50   Output ~ 0
+SWITCH0+
+Text GLabel 2700 1650 1    50   Output ~ 0
+SWITCH0_GND
+Text GLabel 5650 1600 1    50   Input ~ 0
+ADC1
+Text GLabel 6800 1600 1    50   Input ~ 0
+ADC2
+Text GLabel 7900 1600 1    50   Input ~ 0
+ADC3
 $EndSCHEMATC

Commit message: Routing in progress.
Parts:
- removed Q11: IRLML6344TRPBF, symbol Device:Q_NMOS_DGS
- added Q11: IRLML6344TRPBF, Package_TO_SOT_SMD:SOT-23_Handsoldering, symbol Device:Q_NMOS_GSD
- D13: footprint (none) -> Diode_SMD:D_SOT-23_ANK
- D14: footprint (none) -> LED_SMD:LED_0603_1608Metric_Pad1.05x0.95mm_HandSolder
- R50, R51, R52, R53, R54, R55, R56, R57, R58, R59: footprint (none) -> Resistor_SMD:R_0603_1608Metric_Pad1.05x0.95mm_HandSolder
Connections:
- net GND: now also Q11.2 (S)
- net SWITCH0: now also Q11.1 (G)
- net SWITCH0_GND: now also Q11.3 (D)
Changed lines of the file:
@@
 F 0 "R52" H 2230 2904 50  0000 R CNN
 F 1 "10k" H 2230 2995 50  0000 R CNN
-F 2 "" V 2230 2950 50  0001 C CNN
+F 2 "Resistor_SMD:R_0603_1608Metric_Pad1.05x0.95mm_HandSolder" V 2230 2950 50  0001 C CNN
 F 3 "~" H 2300 2950 50  0001 C CNN
 	1    2300 2950
 	-1   0    0    1
-$EndComp
-$Comp
-L Device:Q_NMOS_DGS Q?
-U 1 1 5BEA4E4C
-P 2600 2650
-AR Path="/5BCDDEA6/5BEA4E4C" Ref="Q?"  Part="1"
-AR Path="/5BEA0F8F/5BEA4E4C" Ref="Q11"  Part="1"
-F 0 "Q11" H 2806 2696 50  0000 L CNN
-F 1 "IRLML6344TRPBF" H 2806 2605 50  0000 L CNN
-F 2 "" H 2800 2750 50  0001 C CNN
-F 3 "~" H 2600 2650 50  0001 C CNN
-F 4 "IRLML6344TRPBF" H -2450 -3550 50  0001 C CNN "Farnell"
-F 5 "1857299" H -2450 -3550 50  0001 C CNN "Ref"
-	1    2600 2650
-	1    0    0    -1
 $EndComp
 Wire Wire Line
@@
 F 0 "R50" H 1030 1604 50  0000 R CNN
 F 1 "0" H 1030 1695 50  0000 R CNN
-F 2 "" V 1030 1650 50  0001 C CNN
+F 2 "Resistor_SMD:R_0603_1608Metric_Pad1.05x0.95mm_HandSolder" V 1030 1650 50  0001 C CNN
 F 3 "~" H 1100 1650 50  0001 C CNN
 	1    1100 1650
@@
 F 0 "R51" H 1470 1696 50  0000 L CNN
 F 1 "0" H 1470 1605 50  0000 L CNN
-F 2 "" V 1330 1650 50  0001 C CNN
+F 2 "Resistor_SMD:R_0603_1608Metric_Pad1.05x0.95mm_HandSolder" V 1330 1650 50  0001 C CNN
 F 3 "~" H 1400 1650 50  0001 C CNN
 	1    1400 1650
@@
 F 0 "D13" H 2250 2266 50  0000 C CNN
 F 1 "SBR160S23-7" H 2250 2175 50  0000 C CNN
-F 2 "" H 2250 2050 50  0001 C CNN
+F 2 "Diode_SMD:D_SOT-23_ANK" H 2250 2050 50  0001 C CNN
 F 3 "~" H 2250 2050 50  0001 C CNN
 F 4 "1863724" H -2450 -3550 50  0001 C CNN "Farnell"
@@
 F 0 "D14" V 3488 1382 50  0000 R CNN
 F 1 "LED_GREEN" V 3397 1382 50  0000 R CNN
-F 2 "" H 3450 1500 50  0001 C CNN
+F 2 "LED_SMD:LED_0603_1608Metric_Pad1.05x0.95mm_HandSolder" H 3450 1500 50  0001 C CNN
 F 3 "~" H 3450 1500 50  0001 C CNN
 F 4 "2251490" H -6550 -2650 50  0001 C CNN "Farnell"
@@
 F 0 "R53" H 3380 1804 50  0000 R CNN
 F 1 "1k" H 3380 1895 50  0000 R CNN
-F 2 "" V 3380 1850 50  0001 C CNN
+F 2 "Resistor_SMD:R_0603_1608Metric_Pad1.05x0.95mm_HandSolder" V 3380 1850 50  0001 C CNN
 F 3 "~" H 3450 1850 50  0001 C CNN
 	1    3450 1850
@@
 F 0 "R54" H 5720 1946 50  0000 L CNN
 F 1 "UNKN" H 5720 1855 50  0000 L CNN
-F 2 "" V 5580 1900 50  0001 C CNN
+F 2 "Resistor_SMD:R_0603_1608Metric_Pad1.05x0.95mm_HandSolder" V 5580 1900 50  0001 C CNN
 F 3 "~" H 5650 1900 50  0001 C CNN
 	1    5650 1900
@@
 F 0 "R55" H 5720 2546 50  0000 L CNN
 F 1 "UNKN" H 5720 2455 50  0000 L CNN
-F 2 "" V 5580 2500 50  0001 C CNN
+F 2 "Resistor_SMD:R_0603_1608Metric_Pad1.05x0.95mm_HandSolder" V 5580 2500 50  0001 C CNN
 F 3 "~" H 5650 2500 50  0001 C CNN
 	1    5650 2500
@@
 F 0 "R56" H 6870 1946 50  0000 L CNN
 F 1 "UNKN" H 6870 1855 50  0000 L CNN
-F 2 "" V 6730 1900 50  0001 C CNN
+F 2 "Resistor_SMD:R_0603_1608Metric_Pad1.05x0.95mm_HandSolder" V 6730 1900 50  0001 C CNN
 F 3 "~" H 6800 1900 50  0001 C CNN
 	1    6800 1900
@@
 F 0 "R57" H 6870 2546 50  0000 L CNN
 F 1 "UNKN" H 6870 2455 50  0000 L CNN
-F 2 "" V 6730 2500 50  0001 C CNN
+F 2 "Resistor_SMD:R_0603_1608Metric_Pad1.05x0.95mm_HandSolder" V 6730 2500 50  0001 C CNN
 F 3 "~" H 6800 2500 50  0001 C CNN
 	1    6800 2500
@@
 F 0 "R58" H 7970 1946 50  0000 L CNN
 F 1 "UNKN" H 7970 1855 50  0000 L CNN
-F 2 "" V 7830 1900 50  0001 C CNN
+F 2 "Resistor_SMD:R_0603_1608Metric_Pad1.05x0.95mm_HandSolder" V 7830 1900 50  0001 C CNN
 F 3 "~" H 7900 1900 50  0001 C CNN
 	1    7900 1900
@@
 F 0 "R59" H 7970 2546 50  0000 L CNN
 F 1 "UNKN" H 7970 2455 50  0000 L CNN
-F 2 "" V 7830 2500 50  0001 C CNN
+F 2 "Resistor_SMD:R_0603_1608Metric_Pad1.05x0.95mm_HandSolder" V 7830 2500 50  0001 C CNN
 F 3 "~" H 7900 2500 50  0001 C CNN
 	1    7900 2500
@@
 Text GLabel 7900 1600 1    50   Input ~ 0
 ADC3
+$Comp
+L Device:Q_NMOS_GSD Q?
+U 1 1 5BEC6427
+P 2600 2650
+AR Path="/5BCDDEAC/5BEC6427" Ref="Q?"  Part="1"
+AR Path="/5BCDDEA6/5BEC6427" Ref="Q?"  Part="1"
+AR Path="/5BEA0F8F/5BEC6427" Ref="Q11"  Part="1"
+F 0 "Q11" H 2806 2696 50  0000 L CNN
+F 1 "IRLML6344TRPBF" H 2806 2605 50  0000 L CNN
+F 2 "Package_TO_SOT_SMD:SOT-23_Handsoldering" H 2800 2750 50  0001 C CNN
+F 3 "~" H 2600 2650 50  0001 C CNN
+F 4 "IRLML6344TRPBF" H 750 0   50  0001 C CNN "Farnell"
+F 5 "1857299" H 750 0   50  0001 C CNN "Ref"
+	1    2600 2650
+	1    0    0    -1
+$EndComp
 $EndSCHEMATC
