File: cellar/Microcontroller.sch (KiCad schematic (older format))
At the start: 18 parts, among them J4 PROG, U3 ATxmega64A4U-AU, U4 LM2936-3.3

Commit message: Replaced wirepads by phoenix connectors.
Parts:
- removed J4: PROG, symbol Connector:Conn_01x06_Male
- removed W22: GPIO0, Pads:wirepad_hole_2.2x1mm, symbol pads:WirePad
- removed W23: GPIO1, Pads:wirepad_hole_2.2x1mm, symbol pads:WirePad
- removed W24: GPIO2, Pads:wirepad_hole_2.2x1mm, symbol pads:WirePad
- removed W25: GPIO3, Pads:wirepad_hole_2.2x1mm, symbol pads:WirePad
- removed W26: GPIO4, Pads:wirepad_hole_2.2x1mm, symbol pads:WirePad
- removed W27: GPIO5, Pads:wirepad_hole_2.2x1mm, symbol pads:WirePad
- removed W28: GPIO6, Pads:wirepad_hole_2.2x1mm, symbol pads:WirePad
- removed W29: GPIO7, Pads:wirepad_hole_2.2x1mm, symbol pads:WirePad
- added C19, C20: 15pF/100V, Capacitor_SMD:C_0603_1608Metric_Pad1.05x0.95mm_HandSolder, symbol Device:C
- added Y1: Crystal, Crystal:Crystal_SMD_Abracon_ABM3-2Pin_5.0x3.2mm_HandSoldering, symbol Device:Crystal
- C21: renamed from C25; footprint (none) -> Capacitor_SMD:C_0603_1608Metric_Pad1.05x0.95mm_HandSolder
- C22: renamed from C26; footprint (none) -> Capacitor_SMD:C_0603_1608Metric_Pad1.05x0.95mm_HandSolder
- C23: renamed from C27; footprint (none) -> Capacitor_SMD:C_0603_1608Metric_Pad1.05x0.95mm_HandSolder
- C24: renamed from C23; footprint (none) -> Capacitor_SMD:C_0603_1608Metric_Pad1.05x0.95mm_HandSolder
- C25: renamed from C24; footprint (none) -> Capacitor_Tantalum_SMD:CP_EIA-3216-10_Kemet-I_Pad1.58x1.35mm_HandSolder
- U2: renamed from U3; value ATxmega64A4U-AU -> ATxmega16A4U-AU; symbol MCU_Microchip_ATmega:ATxmega64A4U-AU -> MCU_Microchip_ATmega:ATxmega16A4U-AU; Farnell (none) -> 2066301; Ref (none) -> ATxmega16A4U-AU
- renumbered R52 to R48, R53 to R49, U4 to U3
Connections:
- net labels added: GPIO0, GPIO1, GPIO2, GPIO3, GPIO4
- wire segments 63 -> 67
- no-connect marks 18 -> 17
Other:
- moved on the sheet: C24, C25, U3

Commit message: Routing in progress.
Parts:
- R48, R49: footprint (none) -> Resistor_SMD:R_0603_1608Metric_Pad1.05x0.95mm_HandSolder
Changed lines of the file:
@@
 F 0 "R49" V 4493 1400 50  0000 C CNN
 F 1 "255" V 4584 1400 50  0000 C CNN
-F 2 "" V 4630 1400 50  0001 C CNN
+F 2 "Resistor_SMD:R_0603_1608Metric_Pad1.05x0.95mm_HandSolder" V 4630 1400 50  0001 C CNN
 F 3 "~" H 4700 1400 50  0001 C CNN
 	1    4700 1400
@@
 F 0 "R48" H 2670 2196 50  0000 L CNN
 F 1 "10k" H 2670 2105 50  0000 L CNN
-F 2 "" V 2530 2150 50  0001 C CNN
+F 2 "Resistor_SMD:R_0603_1608Metric_Pad1.05x0.95mm_HandSolder" V 2530 2150 50  0001 C CNN
 F 3 "~" H 2600 2150 50  0001 C CNN
 	1    2600 2150
