File: cellar/Outputs.sch (KiCad schematic (older format))
At the start: 22 parts

Commit message: Schematic done, pending review.
Parts:
- D7: renamed from D?; value LED_RUN -> LED_BLUE; Farnell (none) -> 1581243; Ref (none) -> MCL-S270SBLC
- D8: renamed from D?; value LED_5V-ON -> LED_ORANGE; Farnell (none) -> 5790864; Ref (none) -> HSMD-C170
- D9: renamed from D?; value LED_12V-ON -> LED_RED; Farnell (none) -> 5790839; Ref (none) -> HSMD-C170
- Q10, Q8, Q9: renamed from Q?; Farnell (none) -> IRLML6344TRPBF; Ref (none) -> 1857299
- gave numbers to parts that had none: 16
Connections:
- net labels added: LED_5V-ON_GND, LED_RUN_GND
Other:
- moved on the sheet: D7, D8, D9

Commit message: Replaced wirepads by phoenix connectors.
Parts:
- removed W17: SERVO_PWM, symbol pads:WirePad
- removed W18: SERVO_5V, symbol pads:WirePad
- removed W19: SERVO_GND, symbol pads:WirePad
- removed W20: LED_RUN_GND, symbol pads:WirePad
- removed W21: LED_5V-ON_GND, symbol pads:WirePad
- D10: renamed from D7; Farnell 1581243 -> 2251459; Ref MCL-S270SBLC -> VLMB1300-GS08
- D11: renamed from D8; Farnell 5790864 -> 2251473; Ref HSMD-C170 -> VLMO1300-GS08
- D12: renamed from D9; Farnell 5790839 -> 2251484; Ref HSMD-C170 -> VLMS1300-GS08
- renumbered R34 to R37, R35 to R38, R36 to R39, R37 to R40, R38 to R41, R39 to R42, R40 to R43, R41 to R44, R42 to R45, R43 to R46, R44 to R47
Connections:
- net labels added: SERVO_GND
- net labels removed: SERVO_PWM
- wire segments 55 -> 52
Other:
- moved on the sheet: Q8, R37

Commit message: Routing in progress.
Parts:
- removed Q10, Q9: IRLML6344TRPBF, symbol Device:Q_NMOS_DGS
- added Q10, Q9: IRLML6344TRPBF, Package_TO_SOT_SMD:SOT-23_Handsoldering, symbol Device:Q_NMOS_GSD
- D10, D11, D12: footprint (none) -> LED_SMD:LED_0603_1608Metric_Pad1.05x0.95mm_HandSolder
- Q8: footprint (none) -> Package_TO_SOT_SMD:SOT-23_Handsoldering; symbol Device:Q_NMOS_DGS -> Device:Q_NMOS_GSD
- R37, R38, R39, R40, R41, R42, R43, R44, R45, R46, R47: footprint (none) -> Resistor_SMD:R_0603_1608Metric_Pad1.05x0.95mm_HandSolder
Connections:
- net +3V3: now also Q9.1 (G)
- net GND: now also Q8.2 (S), Q10.2 (S); no longer Q8.3 (S)
- net LED_RUN: now also Q10.1 (G)
- net SERVO_GND: now also Q8.3 (D); no longer Q8.1 (D)
- net SERVO_ON-OFF: now also Q8.1 (G); no longer Q8.2 (G)
- net UART_TX_3V3: now also Q9.2 (S)
- net UART_TX_5V: now also Q9.3 (D)
- net at R43.2, R44.2: now also Q10.3 (D)
Changed lines of the file:
@@
 Servo
 $Comp
-L Device:Q_NMOS_DGS Q8
+L Device:Q_NMOS_GSD Q8
 U 1 1 5BDD36E5
 P 1800 1750
 F 0 "Q8" H 2006 1796 50  0000 L CNN
 F 1 "IRLML6344TRPBF" H 2006 1705 50  0000 L CNN
-F 2 "" H 2000 1850 50  0001 C CNN
+F 2 "Package_TO_SOT_SMD:SOT-23_Handsoldering" H 2000 1850 50  0001 C CNN
 F 3 "~" H 1800 1750 50  0001 C CNN
 F 4 "IRLML6344TRPBF" H -50 -900 50  0001 C CNN "Farnell"
@@
 F 0 "R37" H 1520 1996 50  0000 L CNN
 F 1 "10k" H 1520 1905 50  0000 L CNN
-F 2 "" V 1380 1950 50  0001 C CNN
+F 2 "Resistor_SMD:R_0603_1608Metric_Pad1.05x0.95mm_HandSolder" V 1380 1950 50  0001 C CNN
 F 3 "~" H 1450 1950 50  0001 C CNN
 	1    1450 1950
@@
 	1    0    0    -1
 $EndComp
-$Comp
-L Device:Q_NMOS_DGS Q10
-U 1 1 5BDD450E
-P 5200 2350
-F 0 "Q10" H 5406 2396 50  0000 L CNN
-F 1 "IRLML6344TRPBF" H 4550 2500 50  0000 L CNN
-F 2 "" H 5400 2450 50  0001 C CNN
-F 3 "~" H 5200 2350 50  0001 C CNN
-F 4 "IRLML6344TRPBF" H 0   0   50  0001 C CNN "Farnell"
-F 5 "1857299" H 0   0   50  0001 C CNN "Ref"
-	1    5200 2350
-	1    0    0    -1
-$EndComp
 Wire Wire Line
 	5300 2550 5300 2750
@@
 F 0 "R42" H 4920 2596 50  0000 L CNN
 F 1 "10k" H 4920 2505 50  0000 L CNN
-F 2 "" V 4780 2550 50  0001 C CNN
+F 2 "Resistor_SMD:R_0603_1608Metric_Pad1.05x0.95mm_HandSolder" V 4780 2550 50  0001 C CNN
 F 3 "~" H 4850 2550 50  0001 C CNN
 	1    4850 2550
@@
 F 0 "R44" V 5393 2050 50  0000 C CNN
 F 1 "255" V 5484 2050 50  0000 C CNN
-F 2 "" V 5530 2050 50  0001 C CNN
+F 2 "Resistor_SMD:R_0603_1608Metric_Pad1.05x0.95mm_HandSolder" V 5530 2050 50  0001 C CNN
 F 3 "~" H 5600 2050 50  0001 C CNN
 	1    5600 2050
@@
 F 0 "D10" H 6042 1395 50  0000 C CNN
 F 1 "LED_BLUE" H 6042 1486 50  0000 C CNN
-F 2 "" H 6050 1650 50  0001 C CNN
+F 2 "LED_SMD:LED_0603_1608Metric_Pad1.05x0.95mm_HandSolder" H 6050 1650 50  0001 C CNN
 F 3 "~" H 6050 1650 50  0001 C CNN
 F 4 "2251459" H 0   0   50  0001 C CNN "Farnell"
@@
 F 0 "R43" V 5393 1650 50  0000 C CNN
 F 1 "1k" V 5484 1650 50  0000 C CNN
-F 2 "" V 5530 1650 50  0001 C CNN
+F 2 "Resistor_SMD:R_0603_1608Metric_Pad1.05x0.95mm_HandSolder" V 5530 1650 50  0001 C CNN
 F 3 "~" H 5600 1650 50  0001 C CNN
 	1    5600 1650
@@
 F 0 "R46" V 8793 2000 50  0000 C CNN
 F 1 "255" V 8884 2000 50  0000 C CNN
-F 2 "" V 8930 2000 50  0001 C CNN
+F 2 "Resistor_SMD:R_0603_1608Metric_Pad1.05x0.95mm_HandSolder" V 8930 2000 50  0001 C CNN
 F 3 "~" H 9000 2000 50  0001 C CNN
 	1    9000 2000
@@
 F 0 "D11" H 9442 1295 50  0000 C CNN
 F 1 "LED_ORANGE" H 9442 1386 50  0000 C CNN
-F 2 "" H 9450 1550 50  0001 C CNN
+F 2 "LED_SMD:LED_0603_1608Metric_Pad1.05x0.95mm_HandSolder" H 9450 1550 50  0001 C CNN
 F 3 "~" H 9450 1550 50  0001 C CNN
 F 4 "2251473" H 0   0   50  0001 C CNN "Farnell"
@@
 F 0 "R45" V 8793 1550 50  0000 C CNN
 F 1 "1k" V 8884 1550 50  0000 C CNN
-F 2 "" V 8930 1550 50  0001 C CNN
+F 2 "Resistor_SMD:R_0603_1608Metric_Pad1.05x0.95mm_HandSolder" V 8930 1550 50  0001 C CNN
 F 3 "~" H 9000 1550 50  0001 C CNN
 	1    9000 1550
@@
 F 0 "D12" V 9445 4579 50  0000 L CNN
 F 1 "LED_RED" V 9536 4579 50  0000 L CNN
-F 2 "" H 9500 4500 50  0001 C CNN
+F 2 "LED_SMD:LED_0603_1608Metric_Pad1.05x0.95mm_HandSolder" H 9500 4500 50  0001 C CNN
 F 3 "~" H 9500 4500 50  0001 C CNN
 F 4 "2251484" H 0   0   50  0001 C CNN "Farnell"
@@
 F 0 "R47" H 9430 4904 50  0000 R CNN
 F 1 "4.7k" H 9430 4995 50  0000 R CNN
-F 2 "" V 9430 4950 50  0001 C CNN
+F 2 "Resistor_SMD:R_0603_1608Metric_Pad1.05x0.95mm_HandSolder" V 9430 4950 50  0001 C CNN
 F 3 "~" H 9500 4950 50  0001 C CNN
 	1    9500 4950
@@
 	9500 4350 9500 4200
 $Comp
-L Device:Q_NMOS_DGS Q9
-U 1 1 5BDDAA80
-P 2800 5250
-F 0 "Q9" V 3050 5250 50  0000 C CNN
-F 1 "IRLML6344TRPBF" V 3141 5250 50  0000 C CNN
-F 2 "" H 3000 5350 50  0001 C CNN
-F 3 "~" H 2800 5250 50  0001 C CNN
-F 4 "IRLML6344TRPBF" H 0   0   50  0001 C CNN "Farnell"
-F 5 "1857299" H 0   0   50  0001 C CNN "Ref"
-	1    2800 5250
-	0    1    1    0
-$EndComp
-$Comp
 L Device:R R41
 U 1 1 5BDDAB4B
@@
 F 0 "R41" H 3370 5196 50  0000 L CNN
 F 1 "10k" H 3370 5105 50  0000 L CNN
-F 2 "" V 3230 5150 50  0001 C CNN
+F 2 "Resistor_SMD:R_0603_1608Metric_Pad1.05x0.95mm_HandSolder" V 3230 5150 50  0001 C CNN
 F 3 "~" H 3300 5150 50  0001 C CNN
 	1    3300 5150
@@
 F 0 "R38" H 2370 5196 50  0000 L CNN
 F 1 "10k" H 2370 5105 50  0000 L CNN
-F 2 "" V 2230 5150 50  0001 C CNN
+F 2 "Resistor_SMD:R_0603_1608Metric_Pad1.05x0.95mm_HandSolder" V 2230 5150 50  0001 C CNN
 F 3 "~" H 2300 5150 50  0001 C CNN
 	1    2300 5150
@@
 F 0 "R39" H 2370 6196 50  0000 L CNN
 F 1 "100k" H 2370 6105 50  0000 L CNN
-F 2 "" V 2230 6150 50  0001 C CNN
+F 2 "Resistor_SMD:R_0603_1608Metric_Pad1.05x0.95mm_HandSolder" V 2230 6150 50  0001 C CNN
 F 3 "~" H 2300 6150 50  0001 C CNN
 	1    2300 6150
@@
 F 0 "R40" H 2370 6696 50  0000 L CNN
 F 1 "51k" H 2370 6605 50  0000 L CNN
-F 2 "" V 2230 6650 50  0001 C CNN
+F 2 "Resistor_SMD:R_0603_1608Metric_Pad1.05x0.95mm_HandSolder" V 2230 6650 50  0001 C CNN
 F 3 "~" H 2300 6650 50  0001 C CNN
 	1    2300 6650
@@
 Text GLabel 2450 1450 2    50   Output ~ 0
 SERVO_GND
+$Comp
+L Device:Q_NMOS_GSD Q9
+U 1 1 5BEBF126
+P 2800 5250
+F 0 "Q9" H 3006 5296 50  0000 L CNN
+F 1 "IRLML6344TRPBF" H 3006 5205 50  0000 L CNN
+F 2 "Package_TO_SOT_SMD:SOT-23_Handsoldering" H 3000 5350 50  0001 C CNN
+F 3 "~" H 2800 5250 50  0001 C CNN
+F 4 "IRLML6344TRPBF" H 950 2600 50  0001 C CNN "Farnell"
+F 5 "1857299" H 950 2600 50  0001 C CNN "Ref"
+	1    2800 5250
+	0    1    1    0
+$EndComp
+$Comp
+L Device:Q_NMOS_GSD Q10
+U 1 1 5BEBF1A2
+P 5200 2350
+F 0 "Q10" H 5406 2396 50  0000 L CNN
+F 1 "IRLML6344TRPBF" H 5406 2305 50  0000 L CNN
+F 2 "Package_TO_SOT_SMD:SOT-23_Handsoldering" H 5400 2450 50  0001 C CNN
+F 3 "~" H 5200 2350 50  0001 C CNN
+F 4 "IRLML6344TRPBF" H 3350 -300 50  0001 C CNN "Farnell"
+F 5 "1857299" H 3350 -300 50  0001 C CNN "Ref"
+	1    5200 2350
+	1    0    0    -1
+$EndComp
 $EndSCHEMATC
