File: cellar/Sensors.sch (KiCad schematic (older format))
At the start: 23 parts

Commit message: Schematic done, pending review.
Parts:
- removed U?: MCP3004, symbol Analog_ADC:MCP3004
- C20: renamed from C?; value 0.1uF/25V -> 0.1uF/50V
- Q6: renamed from Q?; Farnell (none) -> IRLML6344TRPBF; Ref (none) -> 1857299
- gave numbers to parts that had none: 20
Connections:
- net labels added: ADC0
- net labels removed: +5V, ADC1, ADC2, ADC3, SPI0_CE, SPI0_MISO, SPI0_MOSI, SPI0_SCLK
- wire segments 76 -> 58
Other:
- note added: "VCOND Measure"
- note removed: "ADC"
- moved on the sheet: C19, C20, Q6, R28, R29, R30

Commit message: Replaced wirepads by phoenix connectors.
Parts:
- removed R27: 4.7k, symbol Device:R
- removed W10: DHT-INT_3V3, symbol pads:WirePad
- removed W11: DHT-INT_GND, symbol pads:WirePad
- removed W12: DHT-EXT_SIG, symbol pads:WirePad
- removed W13: DHT-EXT_3V3, symbol pads:WirePad
- removed W14: DHT-EXT_GND, symbol pads:WirePad
- removed W15: LIGTHSEN_3V3, symbol pads:WirePad
- removed W16: LIGTHSEN_SIG, symbol pads:WirePad
- removed W9: DHT-INT_SIG, symbol pads:WirePad
- added R33: 4.7k, symbol Device:R
- C15: renamed from C20; footprint (none) -> Capacitor_SMD:C_0603_1608Metric_Pad1.05x0.95mm_HandSolder
- C16: renamed from C21; value 0.1uF/25V -> 0.1uF/50V; footprint (none) -> Capacitor_SMD:C_0603_1608Metric_Pad1.05x0.95mm_HandSolder
- C17: renamed from C22; value 0.1uF/25V -> 0.1uF/50V; footprint (none) -> Capacitor_SMD:C_0603_1608Metric_Pad1.05x0.95mm_HandSolder
- C18: renamed from C19; value 0.1uF/25V -> 0.1uF/50V; footprint (none) -> Capacitor_SMD:C_0603_1608Metric_Pad1.05x0.95mm_HandSolder
- renumbered R26 to R29, R28 to R30, R29 to R31, R30 to R32, R31 to R34, R32 to R35, R33 to R36
Connections:
- net labels added: LIGHTSEN_SIG
- wire segments 58 -> 46
Other:
- moved on the sheet: C15, C16, C17, C18, Q6, Q7, R29, R30, R31, R32, R34, R35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

Commit message: Routing in progress.
Parts:
- removed Q6: IRLML6344TRPBF, symbol Device:Q_NMOS_DGS
- added Q6: IRLML6344TRPBF, Package_TO_SOT_SMD:SOT-23_Handsoldering, symbol Device:Q_NMOS_GSD
- Q7: footprint (none) -> Package_TO_SOT_SMD:SOT-23_Handsoldering; symbol Device:Q_NPN_BCE -> Device:Q_NPN_BEC; Farnell (none) -> 2464060; Ref (none) -> MMBT2369LT1G
- R29, R30, R31, R32, R33, R34, R35, R36: footprint (none) -> Resistor_SMD:R_0603_1608Metric_Pad1.05x0.95mm_HandSolder
Connections:
- net GND: now also Q7.2 (E), Q6.2 (S); no longer Q7.3 (E)
- net VCOND_MEASURE: now also Q6.1 (G)
- net at R34.2, R35.1: now also Q7.3 (C); no longer Q7.2 (C)
- net at C15.2, R32.2: now also Q6.3 (D)
Changed lines of the file:
@@
 F 0 "R29" H 1920 1496 50  0000 L CNN
 F 1 "4.7k" H 1920 1405 50  0000 L CNN
-F 2 "" V 1780 1450 50  0001 C CNN
+F 2 "Resistor_SMD:R_0603_1608Metric_Pad1.05x0.95mm_HandSolder" V 1780 1450 50  0001 C CNN
 F 3 "~" H 1850 1450 50  0001 C CNN
 	1    1850 1450
@@
 F 0 "R36" V 8507 1950 50  0000 C CNN
 F 1 "100k" V 8416 1950 50  0000 C CNN
-F 2 "" V 8230 1950 50  0001 C CNN
+F 2 "Resistor_SMD:R_0603_1608Metric_Pad1.05x0.95mm_HandSolder" V 8230 1950 50  0001 C CNN
 F 3 "~" H 8300 1950 50  0001 C CNN
 	1    8300 1950
@@
 $EndComp
 $Comp
-L Device:Q_NPN_BCE Q7
+L Device:Q_NPN_BEC Q7
 U 1 1 5BDA4EF8
 P 7800 1950
 F 0 "Q7" H 7990 1996 50  0000 L CNN
 F 1 "NPN" H 7990 1905 50  0000 L CNN
-F 2 "" H 8000 2050 50  0001 C CNN
+F 2 "Package_TO_SOT_SMD:SOT-23_Handsoldering" H 8000 2050 50  0001 C CNN
 F 3 "~" H 7800 1950 50  0001 C CNN
+F 4 "2464060" H 7800 1950 50  0001 C CNN "Farnell"
+F 5 "MMBT2369LT1G" H 7800 1950 50  0001 C CNN "Ref"
 	1    7800 1950
 	-1   0    0    -1
@@
 F 0 "R34" V 7707 1550 50  0000 C CNN
 F 1 "51k" V 7616 1550 50  0000 C CNN
-F 2 "" V 7430 1550 50  0001 C CNN
+F 2 "Resistor_SMD:R_0603_1608Metric_Pad1.05x0.95mm_HandSolder" V 7430 1550 50  0001 C CNN
 F 3 "~" H 7500 1550 50  0001 C CNN
 	1    7500 1550
@@
 F 0 "R35" V 8507 1550 50  0000 C CNN
 F 1 "10k" V 8416 1550 50  0000 C CNN
-F 2 "" V 8230 1550 50  0001 C CNN
+F 2 "Resistor_SMD:R_0603_1608Metric_Pad1.05x0.95mm_HandSolder" V 8230 1550 50  0001 C CNN
 F 3 "~" H 8300 1550 50  0001 C CNN
 	1    8300 1550
@@
 F 0 "R31" H 3170 4596 50  0000 L CNN
 F 1 "100k" H 3170 4505 50  0000 L CNN
-F 2 "" V 3030 4550 50  0001 C CNN
+F 2 "Resistor_SMD:R_0603_1608Metric_Pad1.05x0.95mm_HandSolder" V 3030 4550 50  0001 C CNN
 F 3 "~" H 3100 4550 50  0001 C CNN
 	1    3100 4550
@@
 F 0 "R32" H 3170 5296 50  0000 L CNN
 F 1 "51k" H 3170 5205 50  0000 L CNN
-F 2 "" V 3030 5250 50  0001 C CNN
+F 2 "Resistor_SMD:R_0603_1608Metric_Pad1.05x0.95mm_HandSolder" V 3030 5250 50  0001 C CNN
 F 3 "~" H 3100 5250 50  0001 C CNN
 	1    3100 5250
@@
 Wire Wire Line
 	3100 4950 3100 5100
-$Comp
-L Device:Q_NMOS_DGS Q?
-U 1 1 5BDF7B40
-P 3000 5800
-AR Path="/5BCDDEA6/5BDF7B40" Ref="Q?"  Part="1"
-AR Path="/5BCDDEA9/5BDF7B40" Ref="Q6"  Part="1"
-F 0 "Q6" H 2900 6050 50  0000 L CNN
-F 1 "IRLML6344TRPBF" H 2350 5950 50  0000 L CNN
-F 2 "" H 3200 5900 50  0001 C CNN
-F 3 "~" H 3000 5800 50  0001 C CNN
-F 4 "IRLML6344TRPBF" H -4450 1850 50  0001 C CNN "Farnell"
-F 5 "1857299" H -4450 1850 50  0001 C CNN "Ref"
-	1    3000 5800
-	1    0    0    -1
-$EndComp
 Wire Wire Line
 	3100 4950 3100 4750
@@
 F 0 "R30" H 2670 6046 50  0000 L CNN
 F 1 "10k" H 2670 5955 50  0000 L CNN
-F 2 "" V 2530 6000 50  0001 C CNN
+F 2 "Resistor_SMD:R_0603_1608Metric_Pad1.05x0.95mm_HandSolder" V 2530 6000 50  0001 C CNN
 F 3 "~" H 2600 6000 50  0001 C CNN
 	1    2600 6000
@@
 F 0 "R33" H 3720 1496 50  0000 L CNN
 F 1 "4.7k" H 3720 1405 50  0000 L CNN
-F 2 "" V 3580 1450 50  0001 C CNN
+F 2 "Resistor_SMD:R_0603_1608Metric_Pad1.05x0.95mm_HandSolder" V 3580 1450 50  0001 C CNN
 F 3 "~" H 3650 1450 50  0001 C CNN
 	1    3650 1450
@@
 Text GLabel 9000 1950 2    50   Input ~ 0
 LIGHTSEN_SIG
+$Comp
+L Device:Q_NMOS_GSD Q?
+U 1 1 5BEBF65E
+P 3000 5800
+AR Path="/5BCDDEAC/5BEBF65E" Ref="Q?"  Part="1"
+AR Path="/5BCDDEA9/5BEBF65E" Ref="Q6"  Part="1"
+F 0 "Q6" H 3206 5846 50  0000 L CNN
+F 1 "IRLML6344TRPBF" H 3206 5755 50  0000 L CNN
+F 2 "Package_TO_SOT_SMD:SOT-23_Handsoldering" H 3200 5900 50  0001 C CNN
+F 3 "~" H 3000 5800 50  0001 C CNN
+F 4 "IRLML6344TRPBF" H 1150 3150 50  0001 C CNN "Farnell"
+F 5 "1857299" H 1150 3150 50  0001 C CNN "Ref"
+	1    3000 5800
+	1    0    0    -1
+$EndComp
 $EndSCHEMATC
