File: cellar/Switches.sch (KiCad schematic (older format))
At the start: 35 parts

Commit message: Schematic done, pending review.
Parts:
- added D10, D11, D13: LED_GREEN, symbol Device:LED
- added R45, R46, R51: 1k, symbol Device:R
- D4, D5, D6: renamed from D?; Farnell (none) -> 1863724; Ref (none) -> SBR160S23-7
- Q1, Q2, Q3, Q4, Q5: renamed from Q?; Farnell (none) -> IRLML6344TRPBF; Ref (none) -> 1857299
- gave numbers to parts that had none: 27
Connections:
- wire segments 112 -> 124
Other:
- moved on the sheet: C16, C17, C18, D4, D5, D6, Q1, Q2, Q3, Q4, Q5, R10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

Commit message: Replaced wirepads by phoenix connectors.
Parts:
- removed W3: HEAT_SWITCH+, Pads:wirepad_hole_2.2x1mm, symbol pads:WirePad
- removed W4: HEAT_SWITCH_GND, Pads:wirepad_hole_2.2x1mm, symbol pads:WirePad
- removed W5: FAN_SWITCH+, Pads:wirepad_hole_2.2x1mm, symbol pads:WirePad
- removed W6: FAN_SWITCH_GND, Pads:wirepad_hole_2.2x1mm, symbol pads:WirePad
- removed W7: DEHUM_SWITCH+, Pads:wirepad_hole_2.2x1mm, symbol pads:WirePad
- removed W8: DEHUM_SWITCH_GND, Pads:wirepad_hole_2.2x1mm, symbol pads:WirePad
- C12: renamed from C16; footprint (none) -> Capacitor_SMD:C_0805_2012Metric_Pad1.15x1.40mm_HandSolder
- C13: renamed from C17; footprint (none) -> Capacitor_SMD:C_0805_2012Metric_Pad1.15x1.40mm_HandSolder
- C14: renamed from C18; footprint (none) -> Capacitor_SMD:C_0805_2012Metric_Pad1.15x1.40mm_HandSolder
- D6: renamed from D10; Farnell 5790852 -> 2251490; Ref HSMG-C170 -> VLMTG1300-GS08
- D7: renamed from D11; Farnell 5790852 -> 2251490; Ref HSMG-C170 -> VLMTG1300-GS08
- D9: renamed from D13; Farnell 5790852 -> 2251490; Ref HSMG-C170 -> VLMTG1300-GS08
- renumbered D6 to D8, R9 to R10, R14 to R13, R13 to R14, R16 to R15, R15 to R16, R18 to R17, R17 to R18, R45 to R20, R46 to R21, R20 to R22, R21 to R23, R22 to R24, R23 to R25, R24 to R26, R25 to R27, R51 to R28, R10 to R9
Connections:
- net labels added: DEHUM_SWITCH+, DEHUM_SWITCH_GND, FAN_SWITCH+, FAN_SWITCH_GND, HEAT_SWITCH+, HEAT_SWITCH_GND

Commit message: Routing in progress.
Parts:
- removed Q1, Q2, Q3, Q4, Q5: IRLML6344TRPBF, symbol Device:Q_NMOS_DGS
- added Q1, Q2, Q3, Q4, Q5: IRLML6344TRPBF, Package_TO_SOT_SMD:SOT-23_Handsoldering, symbol Device:Q_NMOS_GSD
- D4, D5, D8: footprint (none) -> Diode_SMD:D_SOT-23_ANK
- D6, D7, D9: footprint (none) -> LED_SMD:LED_0603_1608Metric_Pad1.05x0.95mm_HandSolder
- R10, R11, R12, R13, R14, R15, R16, R17, R18, R19, R20, R21, R22, R23, R24, R25, R26, R27, R28, R8, R9: footprint (none) -> Resistor_SMD:R_0603_1608Metric_Pad1.05x0.95mm_HandSolder
Connections:
- net DEHUM_LEVER_F: now also Q4.1 (G)
- net DEHUM_SWITCH: now also Q5.1 (G)
- net DEHUM_SWITCH_GND: now also Q4.3 (D), Q5.3 (D)
- net FAN_SWITCH: now also Q3.1 (G)
- net FAN_SWITCH_GND: now also Q3.3 (D)
- net GND: now also Q1.2 (S), Q2.2 (S), Q3.2 (S), Q4.2 (S), Q5.2 (S)
- net HEAT_LEVER_F: now also Q1.1 (G)
- net HEAT_SWITCH: now also Q2.1 (G)
- net HEAT_SWITCH_GND: now also Q1.3 (D), Q2.3 (D)
