File: rpi_power/rpi_power.kicad_pcb (KiCad board)
At the start: 2 copper layers, 69 x 57.4 mm, 68 parts, among them J1 POWER, J2 Raspberry_Pi_2_3, J3 Raspberry_Pi_2_3, J4 ADC, J7 PROG, J9 GPIO, Q10 IRLML6344TRPBF, Q6 IRLML6344TRPBF, U1 TPS54625, U2 ATxmega16A4U-AU, U3 LM2936-3.3, Y1 Crystal

Commit message: Gerber files generated.
Routing:
- net POWER_STATE: track 88.2 -> 92.1 mm
- net BATT+: track 57.0 -> 56.0 mm
- net GND: vias 214 -> 215
Changed lines of the file:
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@@
     (thickness 1.6)
     (drawings 1238)
-    (tracks 681)
+    (tracks 685)
     (zones 0)
     (modules 68)
@@
   (via (at 164.25 87.5) (size 0.8) (drill 0.4) (layers F.Cu B.Cu) (net 2))
   (via (at 164.25 92.5) (size 0.8) (drill 0.4) (layers F.Cu B.Cu) (net 2))
-  (via (at 164.25 97.5) (size 0.8) (drill 0.4) (layers F.Cu B.Cu) (net 2))
-  (via (at 159.25 97.5) (size 0.8) (drill 0.4) (layers F.Cu B.Cu) (net 2))
+  (via (at 163.64 98.06) (size 0.8) (drill 0.4) (layers F.Cu B.Cu) (net 2))
+  (via (at 159.31 98.1) (size 0.8) (drill 0.4) (layers F.Cu B.Cu) (net 2))
   (via (at 159.25 95) (size 0.8) (drill 0.4) (layers F.Cu B.Cu) (net 2))
   (via (at 161.75 95) (size 0.8) (drill 0.4) (layers F.Cu B.Cu) (net 2))
-  (via (at 161.75 97.5) (size 0.8) (drill 0.4) (layers F.Cu B.Cu) (net 2))
+  (via (at 161.69 98.08) (size 0.8) (drill 0.4) (layers F.Cu B.Cu) (net 2))
   (via (at 160.9 77.5) (size 0.8) (drill 0.4) (layers F.Cu B.Cu) (net 2))
   (via (at 157.7 80.8) (size 0.8) (drill 0.4) (layers F.Cu B.Cu) (net 2))
@@
   (via (at 124.17 76.125) (size 0.6) (drill 0.3) (layers F.Cu B.Cu) (net 2))
   (via (at 157.28 118.4) (size 0.8) (drill 0.4) (layers F.Cu B.Cu) (net 2))
+  (via (at 166.29 99.09) (size 0.8) (drill 0.4) (layers F.Cu B.Cu) (net 2))
   (segment (start 165.8 107.1) (end 167.4 107.1) (width 1.2) (layer F.Cu) (net 3) (status 20))
   (segment (start 165.249999 106.549999) (end 165.8 107.1) (width 1.2) (layer F.Cu) (net 3))
@@
   (segment (start 165.17 108.725) (end 168.67 108.725) (width 0.25) (layer F.Cu) (net 28))
   (segment (start 168.67 108.725) (end 169.9 108.725) (width 0.25) (layer B.Cu) (net 28) (status 20))
-  (segment (start 165 108.555) (end 165.17 108.725) (width 0.25) (layer B.Cu) (net 28))
-  (segment (start 165 101.176998) (end 165 108.555) (width 0.25) (layer B.Cu) (net 28))
-  (segment (start 157.126988 100.30001) (end 157.81108 99.615918) (width 0.25) (layer B.Cu) (net 28))
-  (segment (start 137.727008 100.30001) (end 157.126988 100.30001) (width 0.25) (layer B.Cu) (net 28))
   (segment (start 134.4 98.5) (end 135.926998 98.5) (width 0.25) (layer B.Cu) (net 28))
   (segment (start 135.926998 98.5) (end 137.727008 100.30001) (width 0.25) (layer B.Cu) (net 28))
-  (segment (start 163.43892 99.615918) (end 165 101.176998) (width 0.25) (layer B.Cu) (net 28))
-  (segment (start 157.81108 99.615918) (end 163.43892 99.615918) (width 0.25) (layer B.Cu) (net 28))
   (segment (start 170.59 75.42) (end 171.23 76.06) (width 0.25) (layer B.Cu) (net 28))
   (segment (start 170.59 73.52) (end 170.59 75.42) (width 0.25) (layer B.Cu) (net 28))
   (segment (start 170.59 75.42) (end 171.23 76.06) (width 0.25) (layer F.Cu) (net 28))
   (segment (start 170.59 73.525) (end 170.59 75.42) (width 0.25) (layer F.Cu) (net 28))
+  (segment (start 158.584999 98.171344) (end 158.584999 97.525001) (width 0.25) (layer B.Cu) (net 28))
+  (segment (start 137.727008 100.30001) (end 156.456333 100.30001) (width 0.25) (layer B.Cu) (net 28))
+  (segment (start 156.456333 100.30001) (end 158.584999 98.171344) (width 0.25) (layer B.Cu) (net 28))
+  (segment (start 165.17 108.300736) (end 165.17 108.725) (width 0.25) (layer B.Cu) (net 28))
+  (segment (start 165.17 98.516998) (end 165.17 108.300736) (width 0.25) (layer B.Cu) (net 28))
+  (segment (start 163.988001 97.334999) (end 165.17 98.516998) (width 0.25) (layer B.Cu) (net 28))
+  (segment (start 158.775001 97.334999) (end 163.988001 97.334999) (width 0.25) (layer B.Cu) (net 28))
+  (segment (start 158.584999 97.525001) (end 158.775001 97.334999) (width 0.25) (layer B.Cu) (net 28))
   (segment (start 143.476086 109.69574) (end 140.115918 109.69574) (width 0.25) (layer F.Cu) (net 29) (status 20))
   (segment (start 144.580346 110.8) (end 143.476086 109.69574) (width 0.25) (layer F.Cu) (net 29))
@@
   (segment (start 168 104.7) (end 167.36 105.34) (width 1.2) (layer B.Cu) (net 67))
   (segment (start 168 101.8) (end 168 104.7) (width 1.2) (layer B.Cu) (net 67) (status 10))
-  (segment (start 167.45 101.8) (end 168 101.8) (width 0.25) (layer B.Cu) (net 67))
-  (segment (start 164.815908 99.165908) (end 167.45 101.8) (width 0.25) (layer B.Cu) (net 67))
-  (segment (start 156.954025 99.165908) (end 164.815908 99.165908) (width 0.25) (layer B.Cu) (net 67))
-  (segment (start 156.669933 99.45) (end 156.954025 99.165908) (width 0.25) (layer B.Cu) (net 67))
+  (segment (start 156.669933 99.45) (end 158.04 98.079933) (width 0.25) (layer B.Cu) (net 67))
   (segment (start 154.97 99.45) (end 156.669933 99.45) (width 0.25) (layer B.Cu) (net 67))
+  (segment (start 165.98499 96.88499) (end 166.499999 97.399999) (width 0.25) (layer B.Cu) (net 67))
+  (segment (start 158.5886 96.88499) (end 165.98499 96.88499) (width 0.25) (layer B.Cu) (net 67))
+  (segment (start 158.04 97.43359) (end 158.5886 96.88499) (width 0.25) (layer B.Cu) (net 67))
+  (segment (start 158.04 98.079933) (end 158.04 97.43359) (width 0.25) (layer B.Cu) (net 67))
   (zone (net 8) (net_name +5V) (layer F.Cu) (hatch edge 0.508)
     (priority 2)
