File: Power.sch (KiCad schematic (older format))
At the start: 27 parts, among them U1 TPS54625

Commit message: Updated some refs.
Parts:
- R7: value 22.1k 1% -> 22.1k
Changed lines of the file:
@@
 P 7150 3850
 F 0 "R7" H 7220 3896 50  0000 L CNN
-F 1 "22.1k 1%" H 7220 3805 50  0000 L CNN
+F 1 "22.1k" H 7220 3805 50  0000 L CNN
 F 2 "Resistor_SMD:R_0603_1608Metric_Pad1.05x0.95mm_HandSolder" V 7080 3850 50  0001 C CNN
 F 3 "~" H 7150 3850 50  0001 C CNN

Commit message: Minor modifications.
Changed lines of the file:
@@
 Text GLabel 3900 2200 1    50   UnSpc ~ 0
 BATT+
+Wire Wire Line
+	5550 4250 6150 4250
+Connection ~ 5550 4250
+Connection ~ 6150 4250
 $EndSCHEMATC
