File: Board/Connectors.sch (KiCad schematic (older format))
At the start: 6 parts, among them J1 POWER, J2 Raspberry_Pi_2_3, J3 Raspberry_Pi_2_3, J4 ADC, J7 PROG, J9 GPIO

Commit message: Added protection resistors on xmega GPIOs. Corrected prog connector outline.
Parts:
- J7: footprint Connector_PinHeader_2.54mm:PinHeader_2x03_P2.54mm_Vertical -> Connectors_custom:PinHeader_2x03_P2.54mm_Vertical_w_enclosure
Changed lines of the file:
@@
 F 0 "J7" H 10106 5978 50  0000 C CNN
 F 1 "PROG" H 10106 5887 50  0000 C CNN
-F 2 "Connector_PinHeader_2.54mm:PinHeader_2x03_P2.54mm_Vertical" H 10000 5600 50  0001 C CNN
+F 2 "Connectors_custom:PinHeader_2x03_P2.54mm_Vertical_w_enclosure" H 10000 5600 50  0001 C CNN
 F 3 "~" H 10000 5600 50  0001 C CNN
 	1    10000 5600
