File: Board/Sensors.sch (KiCad schematic (older format))
At the start: 14 parts, among them Q6 IRLML6344TRPBF

Commit message: Some mod to track actual board status.
Parts:
- added R14: 4.7k, Resistor_SMD:R_0603_1608Metric_Pad1.05x0.95mm_HandSolder, symbol Device:R
- C15: value 0.1uF/50V -> 10uF/25V
- R31: value 100k -> 37.4k
- R32: value 51k -> 4.7k
Connections:
- net ADC0: now also R14.1
- net at C15.2, Q6.3 (D), R32.2: now also R14.2
Changed lines of the file:
@@
 EESchema Schematic File Version 4
 LIBS:rpi_power-cache
-EELAYER 26 0
+EELAYER 30 0
 EELAYER END
 $Descr A4 11693 8268
@@
 P 2750 3150
 F 0 "R31" H 2820 3196 50  0000 L CNN
-F 1 "100k" H 2820 3105 50  0000 L CNN
+F 1 "37.4k" H 2820 3105 50  0000 L CNN
 F 2 "Resistor_SMD:R_0603_1608Metric_Pad1.05x0.95mm_HandSolder" V 2680 3150 50  0001 C CNN
 F 3 "~" H 2750 3150 50  0001 C CNN
@@
 P 2750 3850
 F 0 "R32" H 2820 3896 50  0000 L CNN
-F 1 "51k" H 2820 3805 50  0000 L CNN
+F 1 "4.7k" H 2820 3805 50  0000 L CNN
 F 2 "Resistor_SMD:R_0603_1608Metric_Pad1.05x0.95mm_HandSolder" V 2680 3850 50  0001 C CNN
 F 3 "~" H 2750 3850 50  0001 C CNN
@@
 P 3100 3850
 F 0 "C15" H 3215 3896 50  0000 L CNN
-F 1 "0.1uF/50V" H 3150 3750 50  0000 L CNN
+F 1 "10uF/25V" H 3150 3750 50  0000 L CNN
 F 2 "Capacitor_SMD:C_0603_1608Metric_Pad1.05x0.95mm_HandSolder" H 3138 3700 50  0001 C CNN
 F 3 "~" H 3100 3850 50  0001 C CNN
@@
 Text GLabel 9300 3200 1    50   Input ~ 0
 ADC3_IN
+$Comp
+L Device:R R14
+U 1 1 5EA5C4C8
+P 2500 3850
+F 0 "R14" H 2250 3900 50  0000 L CNN
+F 1 "4.7k" H 2250 3800 50  0000 L CNN
+F 2 "Resistor_SMD:R_0603_1608Metric_Pad1.05x0.95mm_HandSolder" V 2430 3850 50  0001 C CNN
+F 3 "~" H 2500 3850 50  0001 C CNN
+	1    2500 3850
+	1    0    0    -1
+$EndComp
+Wire Wire Line
+	2500 3700 2500 3550
+Wire Wire Line
+	2500 3550 2750 3550
+Wire Wire Line
+	2500 4000 2500 4100
+Wire Wire Line
+	2500 4100 2750 4100
 $EndSCHEMATC
